File: RGBtoHDMI Amiga Denise CPLD FFC - CDTV Video Slot/RGBtoHDMI Amiga Denise CPLD FFC - CDTV Video Slot - Face Plate.kicad_pcb (KiCad board)
At the start: 2 copper layers, 99 x 40 mm, 6 parts

Commit message: Tweaks
Parts:
- moved solarmon 0.43 mm to (118.1, 95.3)
Routing:
- added copper zone on B.Cu, net (none)
- added copper zone on F.Cu, net (none)
- removed copper zone on B.Cu, net GND
- removed copper zone on F.Cu, net GND
Other:
- outline, holes or cut-outs redrawn
