File: RGBtoHDMI Amiga Denise DIP Breakout FFC - CDTV v2/RGBtoHDMI Amiga Denise DIP Breakout FFC - CDTV v2.sch (KiCad schematic (older format))
At the start: 2 parts

Commit message: Updates
Parts:
- gave numbers to parts that had none: 1
Changed lines of the file:
@@
 Sheet 1 1
 Title "RGBtoHDMI Amiga Denise DIP Breakout - CDTV"
-Date "2021-11-18"
-Rev ""
+Date "2021-12-10"
+Rev "v2"
 Comp ""
 Comment1 ""
@@
 CSYNC
 $Comp
-L Connector_Generic:Conn_02x24_Counter_Clockwise JDenise?
+L Connector_Generic:Conn_02x24_Counter_Clockwise JDenise1
 U 1 1 61B292B4
 P 2250 2625
-F 0 "JDenise?" H 2300 1325 50  0000 C CNN
+F 0 "JDenise1" H 2300 1325 50  0000 C CNN
 F 1 "Conn_02x24_Counter_Clockwise" H 2300 3875 50  0000 C CNN
 F 2 "solarmon_library:DIP-48_W15.24mm_Socket_Turned_Pins" H 2250 2625 50  0001 C CNN
